File: BCD_SSD/BCD_SSD.kicad_pcb (KiCad board)
At the start: 2 copper layers, 61.2 x 31 mm, 148 parts, among them J1 Conn_01x06, J2 Conn_01x07, P1 C5148641, P2 C5148641, P3 C5148641, P4 C5148641, P5 C5148641

Commit message: Theoretically correct decoder
Parts:
- removed the N1 at (60.5, 61.0)
- removed the N1 at (70.6, 61.0)
- removed the N2 at (62.5, 61.0)
- removed the N2 at (72.6, 61.0)
- removed the N3 at (64.5, 61.0)
- removed the N3 at (74.7, 61.0)
- removed the N4 at (66.5, 61.0)
- removed the N4 at (68.6, 61.0)
- removed the N5 at (58.4, 61.0)
- removed the P1 at (60.5, 63.2)
- removed the P1 at (70.6, 63.2)
- removed the P2 at (72.6, 63.2)
- removed the P2 at (62.5, 63.2)
- removed the P3 at (64.5, 63.2)
- removed the P3 at (74.7, 63.2)
- removed the P4 at (66.5, 63.2)
- removed the P4 at (68.6, 63.2)
- removed the P5 at (58.4, 63.2)
- added N1: C2879716, Package_TO_SOT_SMD:SOT-523, F.Cu at (27.6, 66.1)
- added N2: C2879716, Package_TO_SOT_SMD:SOT-523, F.Cu at (29.6, 66.1)
- added N3: C2879716, Package_TO_SOT_SMD:SOT-523, F.Cu at (25.6, 66.1)
- added P1: C5148641, Package_TO_SOT_SMD:SOT-523, F.Cu at (27.6, 68.4)
- added P2: C5148641, Package_TO_SOT_SMD:SOT-523, F.Cu at (29.6, 68.4)
- added P3: C5148641, Package_TO_SOT_SMD:SOT-523, F.Cu at (25.6, 68.4)
Connections:
- N1 pad 1: D -> !D
- N1 pad 1: !D -> D
- N2 pad 1: d3 -> a2
- N3 pad 1: gf1 -> f1
- N3 pad 1: C -> !B
- N3 pad 1: B -> !B
- N3 pad 1: d2 -> a1
- N4 pad 3: f3 -> f1
- P1 pad 1: D -> !D
- P1 pad 1: !D -> D
- P2 pad 1: d3 -> a2
- P3 pad 1: B -> !B
- P3 pad 1: !B -> B
- P3 pad 1: C -> !B
- P3 pad 1: d2 -> a1
- P3 pad 1: gf1 -> f1
- P4 pad 3: f3 -> f1
Routing:
- net a1: track 10.9 -> 60.9 mm, vias 0 -> 4
- net a2: track 10.6 -> 49.3 mm, vias 2 -> 6
- net !A: track 82.5 -> 52.4 mm, vias 6 -> 4
- net f1: track 0.00 -> 21.5 mm, vias 0 -> 2
- net d2: track 19.1 -> 0.00 mm
- net inter: track 204.4 -> 188.8 mm
- net !C: track 99.4 -> 85.0 mm, vias 12 -> 8
- net d3: track 12.7 -> 0.00 mm, vias 2 -> 0
- net !B: track 75.4 -> 86.6 mm, vias 8 -> 10
- net C: track 91.9 -> 102.6 mm, vias 10 -> 9
- net VCC: track 215.8 -> 205.6 mm, vias 65 -> 59
- net B: track 99.3 -> 89.3 mm, vias 12 -> 10
- net !D: track 86.6 -> 77.3 mm, vias 8 -> 6
- net Net-(N2-Pad2): track 31.5 -> 25.2 mm, vias 20 -> 16
- net D: track 107.7 -> 102.8 mm, vias 14 -> 12
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- added copper zone on B.Cu, net GND
- added copper zone on F.Cu, net GND
